Commit message: 将benchmark转变为参数化轨迹

File: src/marl_car_ros2/urdf/simple_marl_car.urdf (robot description, URDF)
Before this commit: robot simple_marl_car, 2 links, 1 joints
Links:
- removed link lidar_link
- added link base_footprint
- added link camera_link; collision box size=0.06 0.05 0.04; visual box size=0.06 0.05 0.04
- added link front_left_wheel_link, mass 0.6; collision cylinder length=0.045 radius=0.055; visual cylinder length=0.045 radius=0.055
- added link front_right_wheel_link, mass 0.6; collision cylinder length=0.045 radius=0.055; visual cylinder length=0.045 radius=0.055
- added link laser_link; collision cylinder length=0.04 radius=0.035; visual cylinder length=0.04 radius=0.035
- added link rear_left_wheel_link, mass 0.6; collision cylinder length=0.045 radius=0.055; visual cylinder length=0.045 radius=0.055
- added link rear_right_wheel_link, mass 0.6; collision cylinder length=0.045 radius=0.055; visual cylinder length=0.045 radius=0.055
- link base_link: geometry collision box size=0.34 0.20 0.12; visual box size=0.25 0.16 0.04
Joints:
- removed joint lidar_joint
- added joint base_footprint_joint: type fixed, parent base_footprint, child base_link, origin xyz=0 0 0.055
- added joint camera_joint: type fixed, parent base_link, child camera_link, origin xyz=0.16 0 0.08
- added joint front_left_wheel_joint: type continuous, parent base_link, child front_left_wheel_link, origin xyz=0.11 0.13 0, axis 0 1 0
- added joint front_right_wheel_joint: type continuous, parent base_link, child front_right_wheel_link, origin xyz=0.11 -0.13 0, axis 0 1 0
- added joint laser_joint: type fixed, parent base_link, child laser_link, origin xyz=0 0 0.195
- added joint rear_left_wheel_joint: type continuous, parent base_link, child rear_left_wheel_link, origin xyz=-0.11 0.13 0, axis 0 1 0
- added joint rear_right_wheel_joint: type continuous, parent base_link, child rear_right_wheel_link, origin xyz=-0.11 -0.13 0, axis 0 1 0
